File: standalone 1-bit logic/standalone_1_bit_logic.sch (EAGLE design)
At the start: 9 parts

Commit message: Removing B and C LEDs since relays have indicator LEDs
Parts:
- removed B_LED, C_LED: (no value), led:LED3MM
Connections:
- net B: no longer B_LED.A
- net C: no longer C_LED.A
- net GNDA: no longer B_LED.C, C_LED.C
Changed lines of the file:
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@@
 </modules>
 <parts>
-<part name="C_LED" library="led" deviceset="LED" device="3MM"/>
-<part name="B_LED" library="led" deviceset="LED" device="3MM"/>
 <part name="XOR_LED" library="led" deviceset="LED" device="3MM"/>
 <part name="OR_LED" library="led" deviceset="LED" device="3MM"/>
@@
 </moduleinsts>
 <instances>
-<instance part="C_LED" gate="G$1" x="40.64" y="45.72"/>
-<instance part="B_LED" gate="G$1" x="40.64" y="68.58" rot="R180"/>
 <instance part="XOR_LED" gate="G$1" x="99.06" y="45.72" rot="R90"/>
 <instance part="OR_LED" gate="G$1" x="99.06" y="53.34" rot="R90"/>
@@
 </segment>
 <segment>
-<wire x1="40.64" y1="73.66" x2="109.22" y2="73.66" width="0.1524" layer="91"/>
-<wire x1="109.22" y1="73.66" x2="109.22" y2="68.58" width="0.1524" layer="91"/>
 <wire x1="109.22" y1="68.58" x2="109.22" y2="60.96" width="0.1524" layer="91"/>
 <wire x1="109.22" y1="60.96" x2="109.22" y2="58.42" width="0.1524" layer="91"/>
 <wire x1="109.22" y1="58.42" x2="109.22" y2="53.34" width="0.1524" layer="91"/>
 <wire x1="109.22" y1="53.34" x2="109.22" y2="45.72" width="0.1524" layer="91"/>
-<wire x1="109.22" y1="45.72" x2="109.22" y2="40.64" width="0.1524" layer="91"/>
-<wire x1="109.22" y1="40.64" x2="40.64" y2="40.64" width="0.1524" layer="91"/>
-<pinref part="B_LED" gate="G$1" pin="C"/>
 <pinref part="NOT_LED" gate="G$1" pin="C"/>
 <wire x1="104.14" y1="68.58" x2="109.22" y2="68.58" width="0.1524" layer="91"/>
-<junction x="109.22" y="68.58"/>
 <pinref part="AND_LED" gate="G$1" pin="C"/>
 <wire x1="104.14" y1="60.96" x2="109.22" y2="60.96" width="0.1524" layer="91"/>
@@
 <pinref part="XOR_LED" gate="G$1" pin="C"/>
 <wire x1="104.14" y1="45.72" x2="109.22" y2="45.72" width="0.1524" layer="91"/>
-<junction x="109.22" y="45.72"/>
-<pinref part="C_LED" gate="G$1" pin="C"/>
 <pinref part="GND2" gate="1" pin="GNDA"/>
 <wire x1="114.3" y1="58.42" x2="109.22" y2="58.42" width="0.1524" layer="91"/>
@@
 <segment>
 <portref moduleinst="LOGIC_BLOCK1" port="B"/>
-<wire x1="40.64" y1="66.04" x2="50.8" y2="66.04" width="0.1524" layer="91"/>
 <junction x="50.8" y="66.04"/>
-<pinref part="B_LED" gate="G$1" pin="A"/>
 <pinref part="B_SWTCH" gate="&gt;PART" pin="S"/>
-<wire x1="27.94" y1="66.04" x2="40.64" y2="66.04" width="0.1524" layer="91"/>
-<junction x="40.64" y="66.04"/>
+<wire x1="27.94" y1="66.04" x2="50.8" y2="66.04" width="0.1524" layer="91"/>
 </segment>
 </net>
@@
 <segment>
 <portref moduleinst="LOGIC_BLOCK1" port="C"/>
-<wire x1="27.94" y1="50.8" x2="40.64" y2="50.8" width="0.1524" layer="91"/>
+<wire x1="27.94" y1="50.8" x2="50.8" y2="50.8" width="0.1524" layer="91"/>
 <junction x="50.8" y="50.8"/>
 <pinref part="C_SWTCH" gate="&gt;PART" pin="S"/>
-<pinref part="C_LED" gate="G$1" pin="A"/>
-<wire x1="40.64" y1="50.8" x2="50.8" y2="50.8" width="0.1524" layer="91"/>
-<wire x1="40.64" y1="50.8" x2="40.64" y2="48.26" width="0.1524" layer="91"/>
-<junction x="40.64" y="50.8"/>
 </segment>
 </net>

Commit message: Adding 1 bit logic block rev B
Connections:
- net +12V: now also C_SWTCH.S; no longer C_SWTCH.P
- net C: now also C_SWTCH.P; no longer C_SWTCH.S
Other:
- moved on the sheet: C_SWTCH
Changed lines of the file:
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@@
 </plain>
 <moduleinsts>
-<moduleinst name="LOGIC_BLOCK1" module="LOGIC_BLOCK" x="71.12" y="58.42"/>
+<moduleinst name="LOGIC_BLOCK1" module="LOGIC_BLOCK" x="66.04" y="58.42"/>
 </moduleinsts>
 <instances>
@@
 <instance part="GND1" gate="1" x="5.08" y="45.72"/>
 <instance part="B_SWTCH" gate="&gt;PART" x="22.86" y="66.04" rot="R270"/>
-<instance part="C_SWTCH" gate="&gt;PART" x="22.86" y="50.8" rot="R270"/>
+<instance part="C_SWTCH" gate="&gt;PART" x="22.86" y="50.8" rot="R90"/>
 <instance part="GND2" gate="1" x="116.84" y="58.42" rot="R90"/>
 <instance part="GND3" gate="1" x="45.72" y="55.88"/>
@@
 <segment>
 <portref moduleinst="LOGIC_BLOCK1" port="NOT"/>
-<wire x1="91.44" y1="66.04" x2="88.9" y2="66.04" width="0.1524" layer="91"/>
 <pinref part="NOT_LED" gate="G$1" pin="A"/>
 <wire x1="96.52" y1="68.58" x2="91.44" y2="68.58" width="0.1524" layer="91"/>
-<wire x1="91.44" y1="68.58" x2="91.44" y2="66.04" width="0.1524" layer="91"/>
-<junction x="91.44" y="66.04"/>
+<wire x1="91.44" y1="68.58" x2="86.36" y2="66.04" width="0.1524" layer="91"/>
 </segment>
 </net>
@@
 <pinref part="GND3" gate="1" pin="GNDA"/>
 <portref moduleinst="LOGIC_BLOCK1" port="GNDA"/>
-<wire x1="45.72" y1="58.42" x2="50.8" y2="58.42" width="0.1524" layer="91"/>
-<junction x="50.8" y="58.42"/>
+<junction x="45.72" y="58.42"/>
 </segment>
 </net>
@@
 <segment>
 <portref moduleinst="LOGIC_BLOCK1" port="B"/>
-<junction x="50.8" y="66.04"/>
+<junction x="45.72" y="66.04"/>
 <pinref part="B_SWTCH" gate="&gt;PART" pin="S"/>
-<wire x1="27.94" y1="66.04" x2="50.8" y2="66.04" width="0.1524" layer="91"/>
-</segment>
-</net>
-<net name="C" class="0">
-<segment>
-<portref moduleinst="LOGIC_BLOCK1" port="C"/>
-<wire x1="27.94" y1="50.8" x2="50.8" y2="50.8" width="0.1524" layer="91"/>
-<junction x="50.8" y="50.8"/>
-<pinref part="C_SWTCH" gate="&gt;PART" pin="S"/>
+<wire x1="27.94" y1="66.04" x2="45.72" y2="66.04" width="0.1524" layer="91"/>
 </segment>
 </net>
@@
 <pinref part="AND_LED" gate="G$1" pin="A"/>
 <portref moduleinst="LOGIC_BLOCK1" port="AND"/>
-<wire x1="91.44" y1="60.96" x2="96.52" y2="60.96" width="0.1524" layer="91"/>
-<junction x="91.44" y="60.96"/>
+<wire x1="86.36" y1="60.96" x2="96.52" y2="60.96" width="0.1524" layer="91"/>
+<junction x="86.36" y="60.96"/>
 </segment>
 </net>
@@
 <pinref part="OR_LED" gate="G$1" pin="A"/>
 <portref moduleinst="LOGIC_BLOCK1" port="OR"/>
-<wire x1="96.52" y1="53.34" x2="91.44" y2="53.34" width="0.1524" layer="91"/>
-<wire x1="91.44" y1="53.34" x2="91.44" y2="55.88" width="0.1524" layer="91"/>
-<junction x="91.44" y="55.88"/>
+<wire x1="96.52" y1="53.34" x2="86.36" y2="55.88" width="0.1524" layer="91"/>
+<junction x="86.36" y="55.88"/>
 </segment>
 </net>
@@
 <pinref part="XOR_LED" gate="G$1" pin="A"/>
 <portref moduleinst="LOGIC_BLOCK1" port="XOR"/>
-<wire x1="91.44" y1="50.8" x2="91.44" y2="45.72" width="0.1524" layer="91"/>
+<wire x1="86.36" y1="50.8" x2="91.44" y2="45.72" width="0.1524" layer="91"/>
 <wire x1="91.44" y1="45.72" x2="96.52" y2="45.72" width="0.1524" layer="91"/>
-<junction x="91.44" y="50.8"/>
+<junction x="86.36" y="50.8"/>
 </segment>
 </net>
@@
 <pinref part="B_SWTCH" gate="&gt;PART" pin="P"/>
 <wire x1="17.78" y1="58.42" x2="17.78" y2="66.04" width="0.1524" layer="91"/>
-<pinref part="C_SWTCH" gate="&gt;PART" pin="P"/>
-<wire x1="17.78" y1="58.42" x2="17.78" y2="50.8" width="0.1524" layer="91"/>
 <junction x="17.78" y="58.42"/>
 <junction x="17.78" y="66.04"/>
 <portref moduleinst="LOGIC_BLOCK1" port="+12V"/>
 <wire x1="17.78" y1="58.42" x2="20.32" y2="60.96" width="0.1524" layer="91"/>
-<wire x1="20.32" y1="60.96" x2="50.8" y2="60.96" width="0.1524" layer="91"/>
-<junction x="50.8" y="60.96"/>
+<wire x1="20.32" y1="60.96" x2="45.72" y2="60.96" width="0.1524" layer="91"/>
+<junction x="45.72" y="60.96"/>
 <pinref part="P+2" gate="1" pin="+12V"/>
 <wire x1="12.7" y1="58.42" x2="17.78" y2="58.42" width="0.1524" layer="91"/>
+<pinref part="C_SWTCH" gate="&gt;PART" pin="S"/>
+<wire x1="17.78" y1="50.8" x2="17.78" y2="58.42" width="0.1524" layer="91"/>
 </segment>
 </net>
+<net name="C" class="0">
+<segment>
+<portref moduleinst="LOGIC_BLOCK1" port="C"/>
+<wire x1="45.72" y1="50.8" x2="27.94" y2="50.8" width="0.1524" layer="91"/>
+<junction x="45.72" y="50.8"/>
+<pinref part="C_SWTCH" gate="&gt;PART" pin="P"/>
+</segment>
+</net>
