File: 4bit ALU/4_bit_ALU.sch (EAGLE design)
At the start: 1 part

Commit message: WIP: 4bit ALU. Input and 3-to-8 decoder
Parts:
- removed PWR: PWR_BLK, relay_computer_custom:PWR_BLK
Connections:
- removed net +12V: PWR-2.K
- removed net GND: PWR-1.K
