File: BBB Connection Test Board/BBBTestCape.sch (EAGLE design)
At the start: 12 parts, among them K1 HF41F-12-H, K2 HF41F-12-H, U1 BTS442E2, U2 BTS442E2, X1 SWTCH_BLCK, X2 SWTCH_BLCK, X3 PWR_BLK, X4 PWR_BLK

Commit message: Finishing BBB Connection Test Board Rev A
Parts:
- removed K1, K2: HF41F-12-H, relay_computer_custom:HF41F-12-H
- removed U1, U2: BTS442E2, relay_computer_custom:BTS442E2
- removed X3, X4: PWR_BLK, relay_computer_custom:PWR_BLK
- LED1, LED2, LED3: OC_NEWARK (none) -> unknown
Connections:
- new net +12V: X1.S, X2.S
- new net BBB1: SV1.1
- new net BBB2: SV1.2
- new net BBB3: SV1.3
- new net BBB4: SV1.4
- new net GND: LED1.C, LED2.C, LED3.C
- new net N$1: LED1.A
- new net N$2: LED3.A, X2.P
- new net N$3: LED2.A, X1.P
Other:
- moved on the sheet: LED1, LED2, LED3, SV1, X1, X2

Commit message: WIP: Starting BBB Connection Test Board rev B. Added MCP23017
Parts:
- removed SV1: (no value), relay_computer_custom:FE04-1
Connections:
- removed net BBB1: SV1.1
- removed net BBB2: SV1.2
- removed net BBB3: SV1.3
- removed net BBB4: SV1.4
Other:
- note added: "HF41F"
- moved on the sheet: LED1, LED2, LED3, X1, X2

Commit message: WIP: starting layout of BBB conn. test board rev B
Parts:
- renumbered LED3 to LED0, X2 to X0
Changed lines of the file:
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@@
 <attribute name="OC_NEWARK" value="unknown"/>
 </part>
-<part name="LED3" library="relay_computer_custom" deviceset="LED" device="3MM">
+<part name="LED0" library="relay_computer_custom" deviceset="LED" device="3MM">
 <attribute name="MF" value=""/>
 <attribute name="MPN" value=""/>
@@
 </part>
 <part name="X1" library="relay_computer_custom" deviceset="SWTCH_BLCK" device=""/>
-<part name="X2" library="relay_computer_custom" deviceset="SWTCH_BLCK" device=""/>
+<part name="X0" library="relay_computer_custom" deviceset="SWTCH_BLCK" device=""/>
 <part name="SUPPLY17" library="supply2" library_urn="urn:adsk.eagle:library:372" deviceset="+12V" device=""/>
 <part name="SUPPLY18" library="supply2" library_urn="urn:adsk.eagle:library:372" deviceset="GND" device=""/>
@@
 <attribute name="MPN" x="58.42" y="99.06" size="1.778" layer="96" rot="R180" display="off"/>
 </instance>
-<instance part="LED3" gate="G$1" x="160.02" y="99.06" rot="R180">
+<instance part="LED0" gate="G$1" x="160.02" y="99.06" rot="R180">
 <attribute name="OC_NEWARK" x="160.02" y="99.06" size="1.778" layer="96" rot="R180" display="off"/>
 <attribute name="MF" x="160.02" y="99.06" size="1.778" layer="96" rot="R180" display="off"/>
@@
 </instance>
 <instance part="X1" gate="&gt;PART" x="50.8" y="91.44" rot="R90"/>
-<instance part="X2" gate="&gt;PART" x="152.4" y="91.44" rot="R90"/>
+<instance part="X0" gate="&gt;PART" x="152.4" y="91.44" rot="R90"/>
 <instance part="SUPPLY17" gate="+12V" x="17.78" y="106.68"/>
 <instance part="SUPPLY18" gate="GND" x="7.62" y="106.68" rot="R180"/>
@@
 <instance part="SUPPLY5" gate="GND" x="129.54" y="83.82" rot="R180"/>
 <instance part="SUPPLY6" gate="+12V" x="121.92" y="83.82"/>
-<instance part="SUPPLY7" gate="GND" x="109.22" y="109.22" rot="R180"/>
+<instance part="SUPPLY7" gate="GND" x="109.22" y="111.76" rot="R180"/>
 <instance part="+3V2" gate="G$1" x="175.26" y="48.26" rot="R180"/>
 <instance part="SUPPLY8" gate="GND" x="175.26" y="83.82" rot="R180"/>
@@
 <pinref part="LED1" gate="G$1" pin="C"/>
 <pinref part="SUPPLY7" gate="GND" pin="GND"/>
-<wire x1="109.22" y1="104.14" x2="109.22" y2="106.68" width="0.1524" layer="91"/>
+<wire x1="109.22" y1="104.14" x2="109.22" y2="109.22" width="0.1524" layer="91"/>
 </segment>
 <segment>
@@
 </segment>
 <segment>
-<pinref part="LED3" gate="G$1" pin="C"/>
+<pinref part="LED0" gate="G$1" pin="C"/>
 <pinref part="SUPPLY9" gate="GND" pin="GND"/>
 <wire x1="160.02" y1="104.14" x2="160.02" y2="109.22" width="0.1524" layer="91"/>
@@
 </segment>
 <segment>
-<pinref part="X2" gate="&gt;PART" pin="S"/>
+<pinref part="X0" gate="&gt;PART" pin="S"/>
 <pinref part="SUPPLY3" gate="+12V" pin="+12V"/>
 <wire x1="144.78" y1="91.44" x2="147.32" y2="91.44" width="0.1524" layer="91"/>
@@
 <net name="N$2" class="0">
 <segment>
-<pinref part="X2" gate="&gt;PART" pin="P"/>
+<pinref part="X0" gate="&gt;PART" pin="P"/>
 <portref moduleinst="12V_TO_3V3_1BIT1" port="IN"/>
 <wire x1="157.48" y1="91.44" x2="160.02" y2="91.44" width="0.1524" layer="91"/>
 <wire x1="160.02" y1="91.44" x2="160.02" y2="81.28" width="0.1524" layer="91"/>
-<pinref part="LED3" gate="G$1" pin="A"/>
+<pinref part="LED0" gate="G$1" pin="A"/>
 <wire x1="160.02" y1="91.44" x2="160.02" y2="96.52" width="0.1524" layer="91"/>
 <junction x="160.02" y="91.44"/>
