File: 4bit Register Board/4bit Register Board.brd (EAGLE design)
At the start: 125 x 140 mm, 161 parts

Commit message: Adding TMP registers back into Register Board
Parts:
- removed OUTPUT_AU_A:X1, OUTPUT_AU_B:X1, OUTPUT_LU_A:X1, OUTPUT_LU_B:X1: 55932-0430, relay_computer_custom:55932-0430
- removed REGISTER_CONTROL:X1: 55932-1230, relay_computer_custom:55932-1230
- added OUTPUT_AU_TMP1:X1, OUTPUT_AU_TMP2:X1, OUTPUT_LU_TMP1:X1, OUTPUT_LU_TMP2:X1: 55932-0430, relay_computer_custom:55932-0430
- added REGISTER_CONTROL:LED_13, REGISTER_CONTROL:LED_14, REGISTER_CONTROL:LED_15, REGISTER_CONTROL:LED_16, REGISTER_CONTROL:LED_17, REGISTER_CONTROL:LED_18, REGISTER_CONTROL:LED_19, REGISTER_CONTROL:LED_20, REGISTER_TMP1:LED0, REGISTER_TMP1:LED1, REGISTER_TMP1:LED2, REGISTER_TMP1:LED3, REGISTER_TMP2:LED0, REGISTER_TMP2:LED1, REGISTER_TMP2:LED2, REGISTER_TMP2:LED3: (no value), relay_computer_custom:LED3MM
- added REGISTER_CONTROL:X2: 55917-2030, relay_computer_custom:55917-2030
- added REGISTER_TMP1:D10, REGISTER_TMP1:D12, REGISTER_TMP1:D14, REGISTER_TMP1:D18, REGISTER_TMP1:D20, REGISTER_TMP1:D4, REGISTER_TMP1:D6, REGISTER_TMP1:D8, REGISTER_TMP1:ENABLE_ADDRESS:D2, REGISTER_TMP1:ENABLE_DATA:D2, REGISTER_TMP2:D10, REGISTER_TMP2:D12, REGISTER_TMP2:D14, REGISTER_TMP2:D18, REGISTER_TMP2:D20, REGISTER_TMP2:D4, REGISTER_TMP2:D6, REGISTER_TMP2:D8, REGISTER_TMP2:ENABLE_ADDRESS:D2, REGISTER_TMP2:ENABLE_DATA:D2: 1N5359, relay_computer_custom:C1702-05
- added REGISTER_TMP1:D11, REGISTER_TMP1:D13, REGISTER_TMP1:D17, REGISTER_TMP1:D19, REGISTER_TMP1:D3, REGISTER_TMP1:D5, REGISTER_TMP1:D7, REGISTER_TMP1:D9, REGISTER_TMP1:ENABLE_ADDRESS:D1, REGISTER_TMP1:ENABLE_DATA:D1, REGISTER_TMP2:D11, REGISTER_TMP2:D13, REGISTER_TMP2:D17, REGISTER_TMP2:D19, REGISTER_TMP2:D3, REGISTER_TMP2:D5, REGISTER_TMP2:D7, REGISTER_TMP2:D9, REGISTER_TMP2:ENABLE_ADDRESS:D1, REGISTER_TMP2:ENABLE_DATA:D1: 1N4007, relay_computer_custom:RAD2,5
- added REGISTER_TMP1:ENABLE_ADDRESS:K1, REGISTER_TMP1:ENABLE_DATA:K1, REGISTER_TMP1:K10, REGISTER_TMP1:K3, REGISTER_TMP2:ENABLE_ADDRESS:K1, REGISTER_TMP2:ENABLE_DATA:K1, REGISTER_TMP2:K10, REGISTER_TMP2:K3: PY14-02, relay_computer_custom:PY14-02
- added REGISTER_TMP1:K2, REGISTER_TMP1:K9, REGISTER_TMP2:K2, REGISTER_TMP2:K9: HF41F-12-Z, relay_computer_custom:HF41F-12-Z
- added REGISTER_TMP1:K4, REGISTER_TMP1:K5, REGISTER_TMP1:K6, REGISTER_TMP1:K7, REGISTER_TMP2:K4, REGISTER_TMP2:K5, REGISTER_TMP2:K6, REGISTER_TMP2:K7: HF41F-12-H, relay_computer_custom:HF41F-12-H
- moved REGISTER_CONTROL:LED_12 551.5 mm to (-195.5, -490.0), turned to 0 degrees
- moved REGISTER_CONTROL:LED_11 539.8 mm to (-161.5, -490.0), turned to 0 degrees
Connections:
- net N$17 renamed LOAD_CCR
- removed net N$6: OUTPUT_AU_B:X1.2, OUTPUT_LU_B:X1.2, REGISTER_B:D9.C, REGISTER_B:ENABLE_ADDRESS:K1.31, REGISTER_B:ENABLE_DATA:K1.21, REGISTER_B:K5.1, REGISTER_B:K5.4, REGISTER_B:LED2.A
- removed net N$7: OUTPUT_AU_B:X1.3, OUTPUT_LU_B:X1.3, REGISTER_B:D11.C, REGISTER_B:ENABLE_ADDRESS:K1.21, REGISTER_B:ENABLE_DATA:K1.31, REGISTER_B:K6.1, REGISTER_B:K6.4, REGISTER_B:LED1.A
- removed net N$8: OUTPUT_AU_B:X1.4, OUTPUT_LU_B:X1.4, REGISTER_B:D13.C, REGISTER_B:ENABLE_ADDRESS:K1.11, REGISTER_B:ENABLE_DATA:K1.41, REGISTER_B:K7.1, REGISTER_B:K7.4, REGISTER_B:LED0.A
- new net LOADA_TMP1: REGISTER_CONTROL:LED_17.A, REGISTER_TMP1:D19.C, REGISTER_TMP1:K10.A2
- new net LOADA_TMP2: REGISTER_CONTROL:LED_19.A, REGISTER_TMP2:D19.C, REGISTER_TMP2:K10.A2
- new net LOADD_TMP1: REGISTER_CONTROL:LED_7.A, REGISTER_CONTROL:X2.13, REGISTER_TMP1:D5.C, REGISTER_TMP1:K3.A2
- new net LOADD_TMP2: REGISTER_CONTROL:LED_9.A, REGISTER_CONTROL:X2.17, REGISTER_TMP2:D5.C, REGISTER_TMP2:K3.A2
- new net N$18: OUTPUT_AU_TMP1:X1.1, OUTPUT_LU_TMP1:X1.1, REGISTER_TMP1:D7.C, REGISTER_TMP1:ENABLE_ADDRESS:K1.41, REGISTER_TMP1:ENABLE_DATA:K1.11, REGISTER_TMP1:K4.1, REGISTER_TMP1:K4.4, REGISTER_TMP1:LED3.A
- new net N$19: OUTPUT_AU_TMP1:X1.2, OUTPUT_LU_TMP1:X1.2, REGISTER_TMP1:D9.C, REGISTER_TMP1:ENABLE_ADDRESS:K1.31, REGISTER_TMP1:ENABLE_DATA:K1.21, REGISTER_TMP1:K5.1, REGISTER_TMP1:K5.4, REGISTER_TMP1:LED2.A
- new net N$20: OUTPUT_AU_TMP1:X1.3, OUTPUT_LU_TMP1:X1.3, REGISTER_TMP1:D11.C, REGISTER_TMP1:ENABLE_ADDRESS:K1.21, REGISTER_TMP1:ENABLE_DATA:K1.31, REGISTER_TMP1:K6.1, REGISTER_TMP1:K6.4, REGISTER_TMP1:LED1.A
- new net N$21: OUTPUT_AU_TMP1:X1.4, OUTPUT_LU_TMP1:X1.4, REGISTER_TMP1:D13.C, REGISTER_TMP1:ENABLE_ADDRESS:K1.11, REGISTER_TMP1:ENABLE_DATA:K1.41, REGISTER_TMP1:K7.1, REGISTER_TMP1:K7.4, REGISTER_TMP1:LED0.A
- new net REGISTER_A:R0: REGISTER_A:D13.C, REGISTER_A:ENABLE_ADDRESS:K1.11, REGISTER_A:ENABLE_DATA:K1.41, REGISTER_A:K7.1, REGISTER_A:K7.4, REGISTER_A:LED0.A
- new net REGISTER_A:R1: REGISTER_A:D11.C, REGISTER_A:ENABLE_ADDRESS:K1.21, REGISTER_A:ENABLE_DATA:K1.31, REGISTER_A:K6.1, REGISTER_A:K6.4, REGISTER_A:LED1.A
- new net REGISTER_A:R2: REGISTER_A:D9.C, REGISTER_A:ENABLE_ADDRESS:K1.31, REGISTER_A:ENABLE_DATA:K1.21, REGISTER_A:K5.1, REGISTER_A:K5.4, REGISTER_A:LED2.A
- new net REGISTER_A:R3: REGISTER_A:D7.C, REGISTER_A:ENABLE_ADDRESS:K1.41, REGISTER_A:ENABLE_DATA:K1.11, REGISTER_A:K4.1, REGISTER_A:K4.4, REGISTER_A:LED3.A
- new net REGISTER_B:R0: REGISTER_B:D13.C, REGISTER_B:ENABLE_ADDRESS:K1.11, REGISTER_B:ENABLE_DATA:K1.41, REGISTER_B:K7.1, REGISTER_B:K7.4, REGISTER_B:LED0.A
- new net REGISTER_B:R1: REGISTER_B:D11.C, REGISTER_B:ENABLE_ADDRESS:K1.21, REGISTER_B:ENABLE_DATA:K1.31, REGISTER_B:K6.1, REGISTER_B:K6.4, REGISTER_B:LED1.A
- new net REGISTER_B:R2: REGISTER_B:D9.C, REGISTER_B:ENABLE_ADDRESS:K1.31, REGISTER_B:ENABLE_DATA:K1.21, REGISTER_B:K5.1, REGISTER_B:K5.4, REGISTER_B:LED2.A
- new net REGISTER_TMP1:D$10: REGISTER_TMP1:D19.A, REGISTER_TMP1:D20.A
- new net REGISTER_TMP1:D$2: REGISTER_TMP1:D3.A, REGISTER_TMP1:D4.A
- new net REGISTER_TMP1:D$3: REGISTER_TMP1:D5.A, REGISTER_TMP1:D6.A
- new net REGISTER_TMP1:D$4: REGISTER_TMP1:D7.A, REGISTER_TMP1:D8.A
- new net REGISTER_TMP1:D$5: REGISTER_TMP1:D10.A, REGISTER_TMP1:D9.A
- new net REGISTER_TMP1:D$6: REGISTER_TMP1:D11.A, REGISTER_TMP1:D12.A
- new net REGISTER_TMP1:D$7: REGISTER_TMP1:D13.A, REGISTER_TMP1:D14.A
- new net REGISTER_TMP1:D$9: REGISTER_TMP1:D17.A, REGISTER_TMP1:D18.A
- new net REGISTER_TMP1:ENABLE_ADDRESS:D$1: REGISTER_TMP1:ENABLE_ADDRESS:D1.A, REGISTER_TMP1:ENABLE_ADDRESS:D2.A
- new net REGISTER_TMP1:ENABLE_DATA:D$1: REGISTER_TMP1:ENABLE_DATA:D1.A, REGISTER_TMP1:ENABLE_DATA:D2.A
- new net REGISTER_TMP1:HOLD: REGISTER_TMP1:K10.32, REGISTER_TMP1:K3.32, REGISTER_TMP1:K4.5, REGISTER_TMP1:K5.5, REGISTER_TMP1:K6.5, REGISTER_TMP1:K7.5
- new net REGISTER_TMP1:IN: REGISTER_TMP1:D3.C, REGISTER_TMP1:K2.1, REGISTER_TMP1:K3.42
- new net REGISTER_TMP1:IN1: REGISTER_TMP1:D17.C, REGISTER_TMP1:K10.42, REGISTER_TMP1:K9.1
- new net REGISTER_TMP2:D$10: REGISTER_TMP2:D19.A, REGISTER_TMP2:D20.A
- new net REGISTER_TMP2:D$2: REGISTER_TMP2:D3.A, REGISTER_TMP2:D4.A
- new net REGISTER_TMP2:D$3: REGISTER_TMP2:D5.A, REGISTER_TMP2:D6.A
- new net REGISTER_TMP2:D$4: REGISTER_TMP2:D7.A, REGISTER_TMP2:D8.A
- new net REGISTER_TMP2:D$5: REGISTER_TMP2:D10.A, REGISTER_TMP2:D9.A
- new net REGISTER_TMP2:D$6: REGISTER_TMP2:D11.A, REGISTER_TMP2:D12.A
- new net REGISTER_TMP2:D$7: REGISTER_TMP2:D13.A, REGISTER_TMP2:D14.A
- new net REGISTER_TMP2:D$9: REGISTER_TMP2:D17.A, REGISTER_TMP2:D18.A
- new net REGISTER_TMP2:ENABLE_ADDRESS:D$1: REGISTER_TMP2:ENABLE_ADDRESS:D1.A, REGISTER_TMP2:ENABLE_ADDRESS:D2.A
- new net REGISTER_TMP2:ENABLE_DATA:D$1: REGISTER_TMP2:ENABLE_DATA:D1.A, REGISTER_TMP2:ENABLE_DATA:D2.A
- new net REGISTER_TMP2:HOLD: REGISTER_TMP2:K10.32, REGISTER_TMP2:K3.32, REGISTER_TMP2:K4.5, REGISTER_TMP2:K5.5, REGISTER_TMP2:K6.5, REGISTER_TMP2:K7.5
- new net REGISTER_TMP2:IN: REGISTER_TMP2:D3.C, REGISTER_TMP2:K2.1, REGISTER_TMP2:K3.42
- new net REGISTER_TMP2:IN1: REGISTER_TMP2:D17.C, REGISTER_TMP2:K10.42, REGISTER_TMP2:K9.1
- new net SELECTA_TMP1: REGISTER_CONTROL:LED_18.A, REGISTER_TMP1:ENABLE_ADDRESS:D1.C, REGISTER_TMP1:ENABLE_ADDRESS:K1.A2, REGISTER_TMP1:K9.3
- new net SELECTA_TMP2: REGISTER_CONTROL:LED_20.A, REGISTER_TMP2:ENABLE_ADDRESS:D1.C, REGISTER_TMP2:ENABLE_ADDRESS:K1.A2, REGISTER_TMP2:K9.3
- new net SELECTD_TMP1: REGISTER_CONTROL:LED_8.A, REGISTER_CONTROL:X2.15, REGISTER_TMP1:ENABLE_DATA:D1.C, REGISTER_TMP1:ENABLE_DATA:K1.A2, REGISTER_TMP1:K2.3
- new net SELECTD_TMP2: REGISTER_CONTROL:LED_10.A, REGISTER_CONTROL:X2.19, REGISTER_TMP2:ENABLE_DATA:D1.C, REGISTER_TMP2:ENABLE_DATA:K1.A2, REGISTER_TMP2:K2.3
- net +12V: now also REGISTER_TMP1:K10.31, REGISTER_TMP1:K10.41, REGISTER_TMP1:K2.4, REGISTER_TMP1:K3.31, REGISTER_TMP1:K3.41, REGISTER_TMP1:K9.4, REGISTER_TMP2:K10.31, REGISTER_TMP2:K10.41, REGISTER_TMP2:K2.4, REGISTER_TMP2:K3.31, REGISTER_TMP2:K3.41, REGISTER_TMP2:K9.4
- net ADDR0: now also REGISTER_TMP1:ENABLE_ADDRESS:K1.14, REGISTER_TMP2:ENABLE_ADDRESS:K1.14
- net ADDR1: now also REGISTER_TMP1:ENABLE_ADDRESS:K1.24, REGISTER_TMP2:ENABLE_ADDRESS:K1.24
- net ADDR2: now also REGISTER_TMP1:ENABLE_ADDRESS:K1.34, REGISTER_TMP2:ENABLE_ADDRESS:K1.34
- net ADDR3: now also REGISTER_TMP1:ENABLE_ADDRESS:K1.44, REGISTER_TMP2:ENABLE_ADDRESS:K1.44
- net DATA0: now also REGISTER_TMP1:ENABLE_DATA:K1.44, REGISTER_TMP2:ENABLE_DATA:K1.44
- net DATA1: now also REGISTER_TMP1:ENABLE_DATA:K1.34, REGISTER_TMP2:ENABLE_DATA:K1.34
- net DATA2: now also REGISTER_TMP1:ENABLE_DATA:K1.24, REGISTER_TMP2:ENABLE_DATA:K1.24
- net DATA3: now also REGISTER_TMP1:ENABLE_DATA:K1.14, REGISTER_TMP2:ENABLE_DATA:K1.14
- net GND: now also REGISTER_CONTROL:LED_13.K, REGISTER_CONTROL:LED_14.K, REGISTER_CONTROL:LED_15.K, REGISTER_CONTROL:LED_16.K, REGISTER_CONTROL:LED_17.K, REGISTER_CONTROL:LED_18.K, REGISTER_CONTROL:LED_19.K, REGISTER_CONTROL:LED_20.K, REGISTER_TMP1:D10.C, REGISTER_TMP1:D12.C, REGISTER_TMP1:D14.C, REGISTER_TMP1:D18.C, REGISTER_TMP1:D20.C, REGISTER_TMP1:D4.C, REGISTER_TMP1:D6.C, REGISTER_TMP1:D8.C, REGISTER_TMP1:ENABLE_ADDRESS:D2.C, REGISTER_TMP1:ENABLE_ADDRESS:K1.A1, REGISTER_TMP1:ENABLE_DATA:D2.C, REGISTER_TMP1:ENABLE_DATA:K1.A1, REGISTER_TMP1:K10.A1, REGISTER_TMP1:K2.2, REGISTER_TMP1:K3.A1, REGISTER_TMP1:K4.2, REGISTER_TMP1:K5.2, REGISTER_TMP1:K6.2, REGISTER_TMP1:K7.2, REGISTER_TMP1:K9.2, REGISTER_TMP1:LED0.K, REGISTER_TMP1:LED1.K, REGISTER_TMP1:LED2.K, REGISTER_TMP1:LED3.K, REGISTER_TMP2:D10.C, REGISTER_TMP2:D12.C, REGISTER_TMP2:D14.C, REGISTER_TMP2:D18.C, REGISTER_TMP2:D20.C, REGISTER_TMP2:D4.C, REGISTER_TMP2:D6.C, REGISTER_TMP2:D8.C, REGISTER_TMP2:ENABLE_ADDRESS:D2.C, REGISTER_TMP2:ENABLE_ADDRESS:K1.A1, REGISTER_TMP2:ENABLE_DATA:D2.C, REGISTER_TMP2:ENABLE_DATA:K1.A1, REGISTER_TMP2:K10.A1, REGISTER_TMP2:K2.2, REGISTER_TMP2:K3.A1, REGISTER_TMP2:K4.2, REGISTER_TMP2:K5.2, REGISTER_TMP2:K6.2, REGISTER_TMP2:K7.2, REGISTER_TMP2:K9.2, REGISTER_TMP2:LED0.K, REGISTER_TMP2:LED1.K, REGISTER_TMP2:LED2.K, REGISTER_TMP2:LED3.K
- net LOADA_A: now also REGISTER_CONTROL:LED_11.A; no longer REGISTER_CONTROL:LED_7.A, REGISTER_CONTROL:X1.7
- net LOADA_B: now also REGISTER_CONTROL:LED_13.A; no longer REGISTER_CONTROL:LED_9.A, REGISTER_CONTROL:X1.9
- net LOADA_C: now also REGISTER_CONTROL:LED_15.A; no longer REGISTER_CONTROL:LED_11.A, REGISTER_CONTROL:X1.11
- net LOADD_A: now also REGISTER_CONTROL:X2.1; no longer REGISTER_CONTROL:X1.1
- net LOADD_B: now also REGISTER_CONTROL:X2.5; no longer REGISTER_CONTROL:X1.3
- net LOADD_C: now also REGISTER_CONTROL:X2.9; no longer REGISTER_CONTROL:X1.5
- net N$1: now also OUTPUT_AU_TMP2:X1.1, OUTPUT_LU_TMP2:X1.1, REGISTER_TMP2:D7.C, REGISTER_TMP2:ENABLE_ADDRESS:K1.41, REGISTER_TMP2:ENABLE_DATA:K1.11, REGISTER_TMP2:K4.1, REGISTER_TMP2:K4.4, REGISTER_TMP2:LED3.A; no longer OUTPUT_AU_A:X1.1, OUTPUT_LU_A:X1.1, REGISTER_A:D7.C, REGISTER_A:ENABLE_ADDRESS:K1.41, REGISTER_A:ENABLE_DATA:K1.11, REGISTER_A:K4.1, REGISTER_A:K4.4, REGISTER_A:LED3.A
- net N$2: now also OUTPUT_AU_TMP2:X1.2, OUTPUT_LU_TMP2:X1.2, REGISTER_TMP2:D9.C, REGISTER_TMP2:ENABLE_ADDRESS:K1.31, REGISTER_TMP2:ENABLE_DATA:K1.21, REGISTER_TMP2:K5.1, REGISTER_TMP2:K5.4, REGISTER_TMP2:LED2.A; no longer OUTPUT_AU_A:X1.2, OUTPUT_LU_A:X1.2, REGISTER_A:D9.C, REGISTER_A:ENABLE_ADDRESS:K1.31, REGISTER_A:ENABLE_DATA:K1.21, REGISTER_A:K5.1, REGISTER_A:K5.4, REGISTER_A:LED2.A
- net N$3: now also OUTPUT_AU_TMP2:X1.3, OUTPUT_LU_TMP2:X1.3, REGISTER_TMP2:D11.C, REGISTER_TMP2:ENABLE_ADDRESS:K1.21, REGISTER_TMP2:ENABLE_DATA:K1.31, REGISTER_TMP2:K6.1, REGISTER_TMP2:K6.4, REGISTER_TMP2:LED1.A; no longer OUTPUT_AU_A:X1.3, OUTPUT_LU_A:X1.3, REGISTER_A:D11.C, REGISTER_A:ENABLE_ADDRESS:K1.21, REGISTER_A:ENABLE_DATA:K1.31, REGISTER_A:K6.1, REGISTER_A:K6.4, REGISTER_A:LED1.A
- net N$4: now also OUTPUT_AU_TMP2:X1.4, OUTPUT_LU_TMP2:X1.4, REGISTER_TMP2:D13.C, REGISTER_TMP2:ENABLE_ADDRESS:K1.11, REGISTER_TMP2:ENABLE_DATA:K1.41, REGISTER_TMP2:K7.1, REGISTER_TMP2:K7.4, REGISTER_TMP2:LED0.A; no longer OUTPUT_AU_A:X1.4, OUTPUT_LU_A:X1.4, REGISTER_A:D13.C, REGISTER_A:ENABLE_ADDRESS:K1.11, REGISTER_A:ENABLE_DATA:K1.41, REGISTER_A:K7.1, REGISTER_A:K7.4, REGISTER_A:LED0.A
- net N$5: no longer OUTPUT_AU_B:X1.1, OUTPUT_LU_B:X1.1
- net SELECTA_A: now also REGISTER_CONTROL:LED_12.A; no longer REGISTER_CONTROL:LED_8.A, REGISTER_CONTROL:X1.8
- net SELECTA_B: now also REGISTER_CONTROL:LED_14.A; no longer REGISTER_CONTROL:LED_10.A, REGISTER_CONTROL:X1.10
- net SELECTA_C: now also REGISTER_CONTROL:LED_16.A; no longer REGISTER_CONTROL:LED_12.A, REGISTER_CONTROL:X1.12
- net SELECTD_A: now also REGISTER_CONTROL:X2.3; no longer REGISTER_CONTROL:X1.2
- net SELECTD_B: now also REGISTER_CONTROL:X2.7; no longer REGISTER_CONTROL:X1.4
- net SELECTD_C: now also REGISTER_CONTROL:X2.11; no longer REGISTER_CONTROL:X1.6

Commit message: Compatibility updates (should be no functional changes)
Parts:
- CCR:D10, CCR:D12, CCR:D14, CCR:D4, CCR:D6, CCR:D8, CCR:ENABLE_DATA:D2, REGISTER_A:D10, REGISTER_A:D12, REGISTER_A:D14, REGISTER_A:D18, REGISTER_A:D20, REGISTER_A:D4, REGISTER_A:D6, REGISTER_A:D8, REGISTER_A:ENABLE_ADDRESS:D2, REGISTER_A:ENABLE_DATA:D2, REGISTER_B:D10, REGISTER_B:D12, REGISTER_B:D14, REGISTER_B:D18, REGISTER_B:D20, REGISTER_B:D4, REGISTER_B:D6, REGISTER_B:D8, REGISTER_B:ENABLE_ADDRESS:D2, REGISTER_B:ENABLE_DATA:D2, REGISTER_C:D10, REGISTER_C:D12, REGISTER_C:D14, REGISTER_C:D18, REGISTER_C:D20, REGISTER_C:D4, REGISTER_C:D6, REGISTER_C:D8, REGISTER_C:ENABLE_ADDRESS:D2, REGISTER_C:ENABLE_DATA:D2, REGISTER_TMP1:D10, REGISTER_TMP1:D12, REGISTER_TMP1:D14, REGISTER_TMP1:D18, REGISTER_TMP1:D20, REGISTER_TMP1:D4, REGISTER_TMP1:D6, REGISTER_TMP1:D8, REGISTER_TMP1:ENABLE_ADDRESS:D2, REGISTER_TMP1:ENABLE_DATA:D2, REGISTER_TMP2:D10, REGISTER_TMP2:D12, REGISTER_TMP2:D14, REGISTER_TMP2:D18, REGISTER_TMP2:D20, REGISTER_TMP2:D4, REGISTER_TMP2:D6, REGISTER_TMP2:D8, REGISTER_TMP2:ENABLE_ADDRESS:D2, REGISTER_TMP2:ENABLE_DATA:D2: value 1N5359 -> 1N5359VERT_SML; device relay_computer_custom:C1702-05 -> relay_computer_custom:RAD2.5_D2
- moved CCR:K7 1799.2 mm to (-27.0, -1555.3)
- moved CCR:D14 1798.4 mm to (-1.27, -1543.8)
- moved CCR:D13 1781.1 mm to (-1.27, -1531.1)
- moved CCR:D12 1761.9 mm to (-1.27, -1508.1)
- moved CCR:D11 1745.0 mm to (-1.27, -1495.4)
- moved CCR:K6 1741.8 mm to (-27.0, -1519.6)
- moved CCR:D10 1725.5 mm to (-1.27, -1472.4)
- moved CCR:D9 1709.0 mm to (-1.27, -1459.7)
- moved CCR:K5 1703.7 mm to (-27.0, -1483.9)
- moved CCR:D8 1689.2 mm to (-1.27, -1436.7)
- moved CCR:D7 1672.9 mm to (-1.27, -1424.0)
- moved CCR:K4 1666.1 mm to (-27.0, -1448.2)
- moved CCR:D6 1663.1 mm to (-1.27, -1411.3)
- moved CCR:D5 1647.2 mm to (-1.27, -1398.6)
- moved CCR:D4 1626.7 mm to (-1.27, -1375.6)
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