File: 4bit Arithmetic Unit/4bit Arithmetic Unit.sch (EAGLE design)
At the start: 0 parts

Commit message: Finishing 4bit AU. Text is actually correct when it appears offset. Worth doing a logical double-check
Changed lines of the file:
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@@
 <module name="INPUT3" prefix="" dx="30.48" dy="20.32">
 <ports>
-<port name="IN0" side="bottom" coord="-7.62" direction="out"/>
+<port name="IN0" side="bottom" coord="7.62" direction="out"/>
 <port name="IN1" side="bottom" coord="0" direction="out"/>
-<port name="IN2" side="bottom" coord="7.62" direction="out"/>
+<port name="IN2" side="bottom" coord="-7.62" direction="out"/>
 <port name="GND" side="left" coord="0" direction="pwr"/>
 </ports>
@@
 <net name="AUE" class="0">
 <segment>
-<portref moduleinst="INPUT3-1" port="IN0"/>
 <label x="121.92" y="114.3" size="1.778" layer="95"/>
 <portref moduleinst="ENABLE4-2" port="ENABLE"/>
@@
 <wire x1="53.34" y1="66.04" x2="53.34" y2="114.3" width="0.1524" layer="91"/>
 <wire x1="53.34" y1="114.3" x2="139.7" y2="114.3" width="0.1524" layer="91"/>
-<wire x1="139.7" y1="114.3" x2="139.7" y2="99.06" width="0.1524" layer="91"/>
 <wire x1="53.34" y1="114.3" x2="-15.24" y2="114.3" width="0.1524" layer="91"/>
 <wire x1="-15.24" y1="114.3" x2="-15.24" y2="66.04" width="0.1524" layer="91"/>
@@
 <label x="-10.16" y="-127" size="1.778" layer="95"/>
 <label x="50.8" y="-111.76" size="1.778" layer="95"/>
+<portref moduleinst="INPUT3-1" port="IN2"/>
+<wire x1="139.7" y1="114.3" x2="139.7" y2="99.06" width="0.1524" layer="91"/>
 </segment>
 </net>
@@
 <net name="SUB" class="0">
 <segment>
-<portref moduleinst="INPUT3-1" port="IN2"/>
-<wire x1="139.7" y1="83.82" x2="129.54" y2="83.82" width="0.1524" layer="91"/>
 <wire x1="129.54" y1="83.82" x2="129.54" y2="-5.08" width="0.1524" layer="91"/>
 <portref moduleinst="SUB_XOR1" port="ENABLE"/>
@@
 <junction x="129.54" y="-5.08"/>
 <label x="119.38" y="-43.18" size="1.778" layer="95"/>
-</segment>
-</net>
+<portref moduleinst="INPUT3-1" port="IN0"/>
+<wire x1="129.54" y1="83.82" x2="139.7" y2="83.82" width="0.1524" layer="91"/>
+</segment>
+</net>

Commit message: Using updated connectors
Changed lines of the file:
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@@
 <instance part="LED1" gate="G$1" x="53.34" y="27.94"/>
 <instance part="LED0" gate="G$1" x="63.5" y="27.94"/>
-<instance part="X1" gate="-2" x="22.86" y="48.26" rot="MR0"/>
-<instance part="X1" gate="-1" x="22.86" y="50.8" rot="MR0"/>
-<instance part="X1" gate="-3" x="22.86" y="45.72" rot="MR0"/>
-<instance part="X1" gate="-4" x="22.86" y="43.18" rot="MR0"/>
+<instance part="X1" gate="-2" x="66.04" y="48.26"/>
+<instance part="X1" gate="-1" x="66.04" y="50.8"/>
+<instance part="X1" gate="-3" x="66.04" y="45.72"/>
+<instance part="X1" gate="-4" x="66.04" y="43.18"/>
 </instances>
 <busses>
@@
 <wire x1="58.42" y1="30.48" x2="63.5" y2="30.48" width="0.1524" layer="91"/>
 <label x="60.96" y="35.56" size="1.778" layer="95" rot="R90"/>
-<wire x1="58.42" y1="30.48" x2="58.42" y2="50.8" width="0.1524" layer="91"/>
+<pinref part="X1" gate="-4" pin="S"/>
+<wire x1="63.5" y1="43.18" x2="58.42" y2="43.18" width="0.1524" layer="91"/>
+<wire x1="58.42" y1="43.18" x2="58.42" y2="30.48" width="0.1524" layer="91"/>
 <junction x="58.42" y="30.48"/>
-<pinref part="X1" gate="-1" pin="S"/>
-<wire x1="25.4" y1="50.8" x2="58.42" y2="50.8" width="0.1524" layer="91"/>
 </segment>
 </net>
@@
 <wire x1="48.26" y1="30.48" x2="53.34" y2="30.48" width="0.1524" layer="91"/>
 <label x="50.8" y="35.56" size="1.778" layer="95" rot="R90"/>
-<wire x1="48.26" y1="48.26" x2="48.26" y2="30.48" width="0.1524" layer="91"/>
+<pinref part="X1" gate="-3" pin="S"/>
+<wire x1="63.5" y1="45.72" x2="48.26" y2="45.72" width="0.1524" layer="91"/>
+<wire x1="48.26" y1="45.72" x2="48.26" y2="30.48" width="0.1524" layer="91"/>
 <junction x="48.26" y="30.48"/>
-<pinref part="X1" gate="-2" pin="S"/>
-<wire x1="25.4" y1="48.26" x2="48.26" y2="48.26" width="0.1524" layer="91"/>
 </segment>
 </net>
@@
 <wire x1="38.1" y1="30.48" x2="43.18" y2="30.48" width="0.1524" layer="91"/>
 <label x="40.64" y="35.56" size="1.778" layer="95" rot="R90"/>
-<wire x1="38.1" y1="45.72" x2="38.1" y2="30.48" width="0.1524" layer="91"/>
+<pinref part="X1" gate="-2" pin="S"/>
+<wire x1="63.5" y1="48.26" x2="38.1" y2="48.26" width="0.1524" layer="91"/>
+<wire x1="38.1" y1="48.26" x2="38.1" y2="30.48" width="0.1524" layer="91"/>
 <junction x="38.1" y="30.48"/>
-<pinref part="X1" gate="-3" pin="S"/>
-<wire x1="25.4" y1="45.72" x2="38.1" y2="45.72" width="0.1524" layer="91"/>
 </segment>
 </net>
@@
 <segment>
 <label x="30.48" y="35.56" size="1.778" layer="95" rot="R90"/>
-<wire x1="27.94" y1="43.18" x2="27.94" y2="30.48" width="0.1524" layer="91"/>
 <pinref part="LED3" gate="G$1" pin="A"/>
 <wire x1="27.94" y1="30.48" x2="27.94" y2="10.16" width="0.1524" layer="91"/>
 <wire x1="27.94" y1="30.48" x2="33.02" y2="30.48" width="0.1524" layer="91"/>
+<pinref part="X1" gate="-1" pin="S"/>
+<wire x1="63.5" y1="50.8" x2="27.94" y2="50.8" width="0.1524" layer="91"/>
+<wire x1="27.94" y1="50.8" x2="27.94" y2="30.48" width="0.1524" layer="91"/>
 <junction x="27.94" y="30.48"/>
-<pinref part="X1" gate="-4" pin="S"/>
-<wire x1="25.4" y1="43.18" x2="27.94" y2="43.18" width="0.1524" layer="91"/>
 </segment>
 </net>
@@
 </plain>
 <instances>
-<instance part="SUPPLY16" gate="GND" x="15.24" y="38.1" rot="R270"/>
-<instance part="LED0" gate="G$1" x="58.42" y="33.02" rot="R180"/>
-<instance part="LED1" gate="G$1" x="48.26" y="33.02" rot="R180"/>
-<instance part="LED2" gate="G$1" x="38.1" y="33.02" rot="R180"/>
-<instance part="LED3" gate="G$1" x="27.94" y="33.02" rot="R180"/>
-<instance part="X1" gate="-2" x="20.32" y="10.16" rot="R180"/>
-<instance part="X1" gate="-1" x="20.32" y="7.62" rot="R180"/>
-<instance part="X1" gate="-3" x="20.32" y="12.7" rot="R180"/>
-<instance part="X1" gate="-4" x="20.32" y="15.24" rot="R180"/>
+<instance part="SUPPLY16" gate="GND" x="-5.08" y="27.94" rot="R270"/>
+<instance part="LED0" gate="G$1" x="38.1" y="22.86" rot="R180"/>
+<instance part="LED1" gate="G$1" x="27.94" y="22.86" rot="R180"/>
+<instance part="LED2" gate="G$1" x="17.78" y="22.86" rot="R180"/>
+<instance part="LED3" gate="G$1" x="7.62" y="22.86" rot="R180"/>
+<instance part="X1" gate="-2" x="50.8" y="7.62" rot="MR180"/>
+<instance part="X1" gate="-1" x="50.8" y="5.08" rot="MR180"/>
+<instance part="X1" gate="-3" x="50.8" y="10.16" rot="MR180"/>
+<instance part="X1" gate="-4" x="50.8" y="12.7" rot="MR180"/>
 </instances>
 <busses>
@@
 <segment>
 <pinref part="LED3" gate="G$1" pin="A"/>
-<wire x1="33.02" y1="30.48" x2="33.02" y2="50.8" width="0.1524" layer="91"/>
-<wire x1="33.02" y1="30.48" x2="27.94" y2="30.48" width="0.1524" layer="91"/>
-<label x="30.48" y="48.26" size="1.778" layer="95" rot="R270"/>
-<wire x1="33.02" y1="30.48" x2="33.02" y2="15.24" width="0.1524" layer="91"/>
-<junction x="33.02" y="30.48"/>
+<wire x1="12.7" y1="20.32" x2="12.7" y2="40.64" width="0.1524" layer="91"/>
+<wire x1="12.7" y1="20.32" x2="7.62" y2="20.32" width="0.1524" layer="91"/>
+<label x="10.16" y="38.1" size="1.778" layer="95" rot="R270"/>
+<pinref part="X1" gate="-1" pin="S"/>
+<wire x1="12.7" y1="20.32" x2="12.7" y2="5.08" width="0.1524" layer="91"/>
+<wire x1="12.7" y1="5.08" x2="48.26" y2="5.08" width="0.1524" layer="91"/>
+<junction x="12.7" y="20.32"/>
+</segment>
+</net>
+<net name="OUT2" class="0">
+<segment>
+<pinref part="LED2" gate="G$1" pin="A"/>
+<wire x1="22.86" y1="20.32" x2="22.86" y2="40.64" width="0.1524" layer="91"/>
+<wire x1="22.86" y1="20.32" x2="17.78" y2="20.32" width="0.1524" layer="91"/>
+<label x="20.32" y="38.1" size="1.778" layer="95" rot="R270"/>
+<pinref part="X1" gate="-2" pin="S"/>
+<wire x1="22.86" y1="20.32" x2="22.86" y2="7.62" width="0.1524" layer="91"/>
+<wire x1="22.86" y1="7.62" x2="48.26" y2="7.62" width="0.1524" layer="91"/>
+<junction x="22.86" y="20.32"/>
+</segment>
+</net>
+<net name="OUT1" class="0">
+<segment>
+<pinref part="LED1" gate="G$1" pin="A"/>
+<wire x1="33.02" y1="20.32" x2="33.02" y2="40.64" width="0.1524" layer="91"/>
+<wire x1="33.02" y1="20.32" x2="27.94" y2="20.32" width="0.1524" layer="91"/>
+<label x="30.48" y="38.1" size="1.778" layer="95" rot="R270"/>
+<pinref part="X1" gate="-3" pin="S"/>
+<wire x1="33.02" y1="20.32" x2="33.02" y2="10.16" width="0.1524" layer="91"/>
+<wire x1="33.02" y1="10.16" x2="48.26" y2="10.16" width="0.1524" layer="91"/>
+<junction x="33.02" y="20.32"/>
+</segment>
+</net>
+<net name="OUT0" class="0">
+<segment>
+<label x="40.64" y="38.1" size="1.778" layer="95" rot="R270"/>
+<pinref part="LED0" gate="G$1" pin="A"/>
+<wire x1="43.18" y1="20.32" x2="43.18" y2="40.64" width="0.1524" layer="91"/>
+<wire x1="43.18" y1="20.32" x2="38.1" y2="20.32" width="0.1524" layer="91"/>
 <pinref part="X1" gate="-4" pin="S"/>
-<wire x1="33.02" y1="15.24" x2="22.86" y2="15.24" width="0.1524" layer="91"/>
-</segment>
-</net>
-<net name="OUT2" class="0">
-<segment>
-<pinref part="LED2" gate="G$1" pin="A"/>
-<wire x1="43.18" y1="30.48" x2="43.18" y2="50.8" width="0.1524" layer="91"/>
-<wire x1="43.18" y1="30.48" x2="38.1" y2="30.48" width="0.1524" layer="91"/>
-<label x="40.64" y="48.26" size="1.778" layer="95" rot="R270"/>
-<pinref part="X1" gate="-3" pin="S"/>
-<wire x1="22.86" y1="12.7" x2="43.18" y2="12.7" width="0.1524" layer="91"/>
-<wire x1="43.18" y1="12.7" x2="43.18" y2="30.48" width="0.1524" layer="91"/>
-<junction x="43.18" y="30.48"/>
-</segment>
-</net>
-<net name="OUT1" class="0">
-<segment>
-<pinref part="LED1" gate="G$1" pin="A"/>
-<wire x1="53.34" y1="30.48" x2="53.34" y2="50.8" width="0.1524" layer="91"/>
-<wire x1="53.34" y1="30.48" x2="48.26" y2="30.48" width="0.1524" layer="91"/>
-<label x="50.8" y="48.26" size="1.778" layer="95" rot="R270"/>
-<pinref part="X1" gate="-2" pin="S"/>
-<wire x1="22.86" y1="10.16" x2="53.34" y2="10.16" width="0.1524" layer="91"/>
-<wire x1="53.34" y1="10.16" x2="53.34" y2="30.48" width="0.1524" layer="91"/>
-<junction x="53.34" y="30.48"/>
-</segment>
-</net>
-<net name="OUT0" class="0">
-<segment>
-<label x="60.96" y="48.26" size="1.778" layer="95" rot="R270"/>
-<pinref part="X1" gate="-1" pin="S"/>
-<wire x1="22.86" y1="7.62" x2="63.5" y2="7.62" width="0.1524" layer="91"/>
-<wire x1="63.5" y1="7.62" x2="63.5" y2="30.48" width="0.1524" layer="91"/>
-<pinref part="LED0" gate="G$1" pin="A"/>
-<wire x1="63.5" y1="30.48" x2="63.5" y2="50.8" width="0.1524" layer="91"/>
-<wire x1="63.5" y1="30.48" x2="58.42" y2="30.48" width="0.1524" layer="91"/>
-<junction x="63.5" y="30.48"/>
+<wire x1="43.18" y1="20.32" x2="43.18" y2="12.7" width="0.1524" layer="91"/>
+<wire x1="43.18" y1="12.7" x2="48.26" y2="12.7" width="0.1524" layer="91"/>
+<junction x="43.18" y="20.32"/>
 </segment>
 </net>
@@
 <segment>
 <pinref part="SUPPLY16" gate="GND" pin="GND"/>
-<wire x1="17.78" y1="38.1" x2="38.1" y2="38.1" width="0.1524" layer="91"/>
+<wire x1="-2.54" y1="27.94" x2="17.78" y2="27.94" width="0.1524" layer="91"/>
 <pinref part="LED0" gate="G$1" pin="C"/>
 <pinref part="LED1" gate="G$1" pin="C"/>
-<wire x1="58.42" y1="38.1" x2="48.26" y2="38.1" width="0.1524" layer="91"/>
-<junction x="58.42" y="38.1"/>
+<wire x1="38.1" y1="27.94" x2="27.94" y2="27.94" width="0.1524" layer="91"/>
+<junction x="38.1" y="27.94"/>
 <pinref part="LED2" gate="G$1" pin="C"/>
-<wire x1="48.26" y1="38.1" x2="38.1" y2="38.1" width="0.1524" layer="91"/>
-<junction x="48.26" y="38.1"/>
+<wire x1="27.94" y1="27.94" x2="17.78" y2="27.94" width="0.1524" layer="91"/>
+<junction x="27.94" y="27.94"/>
 <pinref part="LED3" gate="G$1" pin="C"/>
-<wire x1="38.1" y1="38.1" x2="27.94" y2="38.1" width="0.1524" layer="91"/>
-<junction x="38.1" y="38.1"/>
+<wire x1="17.78" y1="27.94" x2="7.62" y2="27.94" width="0.1524" layer="91"/>
+<junction x="17.78" y="27.94"/>
 </segment>
 </net>
@@
 <label x="50.8" y="-111.76" size="1.778" layer="95"/>
 <portref moduleinst="INPUT3-1" port="IN2"/>
-<wire x1="139.7" y1="114.3" x2="139.7" y2="99.06" width="0.1524" layer="91"/>
-</segment>
-</net>
+<wire x1="139.7" y1="99.06" x2="139.7" y2="114.3" width="0.1524" layer="91"/>
+</segment>
+</net>

Commit message: Minor formatting changes
Changed lines of the file:
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@@
 <moduleinst name="ADDER8-1" module="ADDER8" x="50.8" y="-43.18"/>
 <moduleinst name="ZERO_DETECT1" module="ZERO_DETECT" x="45.72" y="-81.28" rot="R270"/>
-<moduleinst name="OUTPUT4-1" module="OUTPUT4" x="78.74" y="-170.18"/>
+<moduleinst name="OUTPUT4-1" module="OUTPUT4" x="78.74" y="-167.64"/>
 <moduleinst name="OUTPUT4-2" module="OUTPUT4" x="25.4" y="-167.64"/>
 <moduleinst name="ENABLE4-3" module="ENABLE4" x="25.4" y="-132.08"/>
@@
 <instance part="SUPPLY12" gate="GND" x="53.34" y="-104.14" rot="R90"/>
 <instance part="SUPPLY10" gate="GND" x="-2.54" y="-43.18" rot="R270"/>
-<instance part="SUPPLY11" gate="GND" x="55.88" y="-170.18" rot="R270"/>
+<instance part="SUPPLY11" gate="GND" x="55.88" y="-167.64" rot="R270"/>
 <instance part="SUPPLY14" gate="GND" x="2.54" y="-167.64" rot="R270"/>
 <instance part="SUPPLY15" gate="+12V" x="-2.54" y="-38.1" rot="R90"/>
@@
 <portref moduleinst="ENABLE4-4" port="OUT3"/>
 <portref moduleinst="OUTPUT4-1" port="OUT3"/>
-<wire x1="66.04" y1="-154.94" x2="66.04" y2="-147.32" width="0.1524" layer="91"/>
+<wire x1="66.04" y1="-152.4" x2="66.04" y2="-147.32" width="0.1524" layer="91"/>
 <label x="63.5" y="-152.4" size="1.778" layer="95" rot="R90"/>
 </segment>
@@
 <portref moduleinst="ENABLE4-4" port="OUT2"/>
 <portref moduleinst="OUTPUT4-1" port="OUT2"/>
-<wire x1="73.66" y1="-154.94" x2="73.66" y2="-147.32" width="0.1524" layer="91"/>
+<wire x1="73.66" y1="-152.4" x2="73.66" y2="-147.32" width="0.1524" layer="91"/>
 <label x="71.12" y="-152.4" size="1.778" layer="95" rot="R90"/>
 </segment>
@@
 <portref moduleinst="ENABLE4-4" port="OUT1"/>
 <portref moduleinst="OUTPUT4-1" port="OUT1"/>
-<wire x1="81.28" y1="-154.94" x2="81.28" y2="-147.32" width="0.1524" layer="91"/>
+<wire x1="81.28" y1="-152.4" x2="81.28" y2="-147.32" width="0.1524" layer="91"/>
 <label x="78.74" y="-152.4" size="1.778" layer="95" rot="R90"/>
 </segment>
@@
 <portref moduleinst="ENABLE4-4" port="OUT0"/>
 <portref moduleinst="OUTPUT4-1" port="OUT0"/>
-<wire x1="88.9" y1="-154.94" x2="88.9" y2="-147.32" width="0.1524" layer="91"/>
+<wire x1="88.9" y1="-152.4" x2="88.9" y2="-147.32" width="0.1524" layer="91"/>
 <label x="86.36" y="-152.4" size="1.778" layer="95" rot="R90"/>
 </segment>

Commit message: The AU opcode wires were switched
Changed lines of the file:
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@@
 <?xml version="1.0" encoding="utf-8"?>
 <!DOCTYPE eagle SYSTEM "eagle.dtd">
-<eagle version="8.3.2">
+<eagle version="8.7.0">
 <drawing>
 <settings>
@@
 <moduleinst name="INPUT4-1" module="INPUT4" x="35.56" y="99.06"/>
 <moduleinst name="INPUT4-2" module="INPUT4" x="78.74" y="99.06"/>
-<moduleinst name="INPUT3-1" module="INPUT3" x="154.94" y="91.44" rot="R270"/>
+<moduleinst name="INPUT3-1" module="INPUT3" x="124.46" y="99.06"/>
 <moduleinst name="ENABLE4-1" module="ENABLE4" x="35.56" y="63.5"/>
 <moduleinst name="ENABLE4-2" module="ENABLE4" x="78.74" y="63.5"/>
@@
 <instance part="SUPPLY2" gate="GND" x="15.24" y="101.6" rot="R180"/>
 <instance part="SUPPLY4" gate="GND" x="58.42" y="101.6" rot="R180"/>
-<instance part="SUPPLY1" gate="GND" x="154.94" y="111.76" rot="R180"/>
+<instance part="SUPPLY1" gate="GND" x="104.14" y="101.6" rot="R180"/>
 <instance part="SUPPLY3" gate="GND" x="58.42" y="58.42"/>
 <instance part="SUPPLY5" gate="GND" x="15.24" y="58.42"/>
@@
 <portref moduleinst="INPUT3-1" port="GND"/>
 <pinref part="SUPPLY1" gate="GND" pin="GND"/>
-<wire x1="154.94" y1="111.76" x2="154.94" y2="109.22" width="0.1524" layer="91"/>
 </segment>
 <segment>
@@
 <net name="AUE" class="0">
 <segment>
-<label x="121.92" y="114.3" size="1.778" layer="95"/>
 <portref moduleinst="ENABLE4-2" port="ENABLE"/>
 <wire x1="58.42" y1="66.04" x2="53.34" y2="66.04" width="0.1524" layer="91"/>
 <wire x1="53.34" y1="66.04" x2="53.34" y2="114.3" width="0.1524" layer="91"/>
-<wire x1="53.34" y1="114.3" x2="139.7" y2="114.3" width="0.1524" layer="91"/>
 <wire x1="53.34" y1="114.3" x2="-15.24" y2="114.3" width="0.1524" layer="91"/>
 <wire x1="-15.24" y1="114.3" x2="-15.24" y2="66.04" width="0.1524" layer="91"/>
-<junction x="53.34" y="114.3"/>
 <portref moduleinst="ENABLE4-1" port="ENABLE"/>
 <wire x1="-15.24" y1="66.04" x2="15.24" y2="66.04" width="0.1524" layer="91"/>
@@
 <label x="-10.16" y="-127" size="1.778" layer="95"/>
 <label x="50.8" y="-111.76" size="1.778" layer="95"/>
+<wire x1="53.34" y1="114.3" x2="99.06" y2="114.3" width="0.1524" layer="91"/>
+<wire x1="99.06" y1="114.3" x2="99.06" y2="83.82" width="0.1524" layer="91"/>
+<junction x="53.34" y="114.3"/>
 <portref moduleinst="INPUT3-1" port="IN2"/>
-<wire x1="139.7" y1="99.06" x2="139.7" y2="114.3" width="0.1524" layer="91"/>
+<wire x1="116.84" y1="83.82" x2="99.06" y2="83.82" width="0.1524" layer="91"/>
+<label x="93.98" y="111.76" size="1.778" layer="95"/>
 </segment>
 </net>
@@
 <net name="INC/DEC" class="0">
 <segment>
-<portref moduleinst="INPUT3-1" port="IN1"/>
 <portref moduleinst="INC/DEC_FILTER1" port="ENABLE"/>
-<wire x1="139.7" y1="91.44" x2="101.6" y2="91.44" width="0.1524" layer="91"/>
-<wire x1="101.6" y1="91.44" x2="101.6" y2="25.4" width="0.1524" layer="91"/>
-<label x="119.38" y="91.44" size="1.778" layer="95"/>
+<wire x1="132.08" y1="25.4" x2="101.6" y2="25.4" width="0.1524" layer="91"/>
+<label x="104.14" y="27.94" size="1.778" layer="95"/>
+<portref moduleinst="INPUT3-1" port="IN0"/>
+<wire x1="132.08" y1="25.4" x2="132.08" y2="83.82" width="0.1524" layer="91"/>
 </segment>
 </net>
@@
 <net name="SUB" class="0">
 <segment>
-<wire x1="129.54" y1="83.82" x2="129.54" y2="-5.08" width="0.1524" layer="91"/>
+<wire x1="124.46" y1="83.82" x2="124.46" y2="-5.08" width="0.1524" layer="91"/>
 <portref moduleinst="SUB_XOR1" port="ENABLE"/>
-<wire x1="129.54" y1="-5.08" x2="101.6" y2="-5.08" width="0.1524" layer="91"/>
-<label x="119.38" y="-5.08" size="1.778" layer="95"/>
+<wire x1="124.46" y1="-5.08" x2="101.6" y2="-5.08" width="0.1524" layer="91"/>
+<label x="104.14" y="-2.54" size="1.778" layer="95"/>
 <portref moduleinst="ADDER8-1" port="CIN"/>
-<wire x1="129.54" y1="-5.08" x2="129.54" y2="-43.18" width="0.1524" layer="91"/>
-<wire x1="129.54" y1="-43.18" x2="101.6" y2="-43.18" width="0.1524" layer="91"/>
-<junction x="129.54" y="-5.08"/>
-<label x="119.38" y="-43.18" size="1.778" layer="95"/>
-<portref moduleinst="INPUT3-1" port="IN0"/>
-<wire x1="129.54" y1="83.82" x2="139.7" y2="83.82" width="0.1524" layer="91"/>
-</segment>
-</net>
+<wire x1="124.46" y1="-5.08" x2="124.46" y2="-43.18" width="0.1524" layer="91"/>
+<wire x1="124.46" y1="-43.18" x2="101.6" y2="-43.18" width="0.1524" layer="91"/>
+<junction x="124.46" y="-5.08"/>
+<label x="104.14" y="-40.64" size="1.778" layer="95"/>
+</segment>
+</net>
