File: 4bit Logic Unit/4bit Logic Unit.sch (EAGLE design)
At the start: 0 parts

Commit message: Minor formatting changes
Changed lines of the file:
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@@
 <?xml version="1.0" encoding="utf-8"?>
 <!DOCTYPE eagle SYSTEM "eagle.dtd">
-<eagle version="8.3.2">
+<eagle version="8.4.3">
 <drawing>
 <settings>
@@
 </segment>
 </net>
-<net name="NOT" class="0">
+<net name="XOR" class="0">
 <segment>
 <pinref part="K2" gate="4" pin="O"/>
@@
 </segment>
 </net>
-<net name="XOR" class="0">
+<net name="NOT" class="0">
 <segment>
 <pinref part="K2" gate="5" pin="S"/>
@@
 <wire x1="30.48" y1="43.18" x2="30.48" y2="22.86" width="0.1524" layer="91"/>
 <wire x1="30.48" y1="22.86" x2="86.36" y2="22.86" width="0.1524" layer="91"/>
-<label x="86.36" y="22.86" size="1.778" layer="95"/>
+<label x="83.82" y="22.86" size="1.778" layer="95"/>
 </segment>
 </net>
@@
 <moduleinst name="ENABLE_B" module="ENABLE4" x="78.74" y="63.5"/>
 <moduleinst name="ZERO_DETECT1" module="ZERO_DETECT" x="45.72" y="-27.94" rot="R270"/>
-<moduleinst name="OUTPUT4-1" module="OUTPUT4" x="78.74" y="-116.84"/>
+<moduleinst name="OUTPUT4-1" module="OUTPUT4" x="78.74" y="-114.3"/>
 <moduleinst name="OUTPUT4-2" module="OUTPUT4" x="25.4" y="-114.3"/>
 <moduleinst name="ENABLE4-3" module="ENABLE4" x="25.4" y="-78.74"/>
@@
 <instance part="SUPPLY13" gate="+12V" x="45.72" y="-50.8" rot="R90"/>
 <instance part="SUPPLY12" gate="GND" x="53.34" y="-50.8" rot="R90"/>
-<instance part="SUPPLY11" gate="GND" x="55.88" y="-116.84" rot="R270"/>
+<instance part="SUPPLY11" gate="GND" x="55.88" y="-114.3" rot="R270"/>
 <instance part="SUPPLY14" gate="GND" x="2.54" y="-114.3" rot="R270"/>
 <instance part="SUPPLY16" gate="GND" x="2.54" y="-81.28" rot="R270"/>
@@
 <wire x1="58.42" y1="-58.42" x2="58.42" y2="-76.2" width="0.1524" layer="91"/>
 <junction x="-2.54" y="-58.42"/>
-<label x="-10.16" y="-73.66" size="1.778" layer="95"/>
-<label x="53.34" y="-60.96" size="1.778" layer="95"/>
+<label x="0" y="-73.66" size="1.778" layer="95"/>
+<label x="53.34" y="-73.66" size="1.778" layer="95"/>
 <wire x1="96.52" y1="114.3" x2="96.52" y2="83.82" width="0.1524" layer="91"/>
 <portref moduleinst="INPUT_OP" port="IN2"/>
@@
 <portref moduleinst="ENABLE4-4" port="OUT3"/>
 <portref moduleinst="OUTPUT4-1" port="OUT3"/>
-<wire x1="66.04" y1="-101.6" x2="66.04" y2="-93.98" width="0.1524" layer="91"/>
+<wire x1="66.04" y1="-99.06" x2="66.04" y2="-93.98" width="0.1524" layer="91"/>
 <label x="63.5" y="-99.06" size="1.778" layer="95" rot="R90"/>
 </segment>
@@
 <portref moduleinst="ENABLE4-4" port="OUT2"/>
 <portref moduleinst="OUTPUT4-1" port="OUT2"/>
-<wire x1="73.66" y1="-101.6" x2="73.66" y2="-93.98" width="0.1524" layer="91"/>
+<wire x1="73.66" y1="-99.06" x2="73.66" y2="-93.98" width="0.1524" layer="91"/>
 <label x="71.12" y="-99.06" size="1.778" layer="95" rot="R90"/>
 </segment>
@@
 <portref moduleinst="ENABLE4-4" port="OUT1"/>
 <portref moduleinst="OUTPUT4-1" port="OUT1"/>
-<wire x1="81.28" y1="-101.6" x2="81.28" y2="-93.98" width="0.1524" layer="91"/>
+<wire x1="81.28" y1="-99.06" x2="81.28" y2="-93.98" width="0.1524" layer="91"/>
 <label x="78.74" y="-99.06" size="1.778" layer="95" rot="R90"/>
 </segment>
@@
 <portref moduleinst="ENABLE4-4" port="OUT0"/>
 <portref moduleinst="OUTPUT4-1" port="OUT0"/>
-<wire x1="88.9" y1="-101.6" x2="88.9" y2="-93.98" width="0.1524" layer="91"/>
+<wire x1="88.9" y1="-99.06" x2="88.9" y2="-93.98" width="0.1524" layer="91"/>
 <label x="86.36" y="-99.06" size="1.778" layer="95" rot="R90"/>
 </segment>
